Commit message: using ros2_control

File: src/neobot/urdf/neobot_description.urdf (robot description, URDF)
Before this commit: robot neobot, 9 links, 8 joints
Links:
- link base_link: geometry collision mesh filename=/home/akarsh/neobot_ws/src/neobot/meshes/base_link.STL; visual mesh filename=/home/akarsh/neobot_ws/src/neobot/meshes/base_link.STL
- link front_castor_link: geometry collision mesh filename=/home/akarsh/neobot_ws/src/neobot/meshes/front_castor_link.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; visual mesh filename=/home/akarsh/neobot_ws/src/neobot/meshes/front_castor_link.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
- link left_wheel_link: geometry collision mesh filename=/home/akarsh/neobot_ws/src/neobot/meshes/left_wheel_link.STL; visual mesh filename=/home/akarsh/neobot_ws/src/neobot/meshes/left_wheel_link.STL
- link rear_castor_link: geometry collision mesh filename=/home/akarsh/neobot_ws/src/neobot/meshes/rear_castor_link.S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; visual mesh filename=/home/akarsh/neobot_ws/src/neobot/meshes/rear_castor_link.S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
- link right_wheel_link: geometry collision mesh filename=/home/akarsh/neobot_ws/src/neobot/meshes/right_wheel_link.S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; visual mesh filename=/home/akarsh/neobot_ws/src/neobot/meshes/right_wheel_link.S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
